File: lightup-namebadge.kicad_pcb (KiCad board)
At the start: 2 copper layers, 100 x 50 mm, 26 parts, among them Q1 PNP, Q2 NPN, Q3 NPN, Q4 NPN, Q5 NPN, SW1 SW_Push, SW2 SW_Push

Commit message: fix: disconnect pin 3 of RV1 from VSS to save power
Connections:
- RV1 pad 3: VSS -> unconnected-(RV1-Pad3)
Routing:
- net VSS: track 80.5 -> 70.5 mm
Changed lines of the file:
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@@
 	(net 12 "Net-(Q2-E)")
 	(net 13 "LEDS_INPUT")
+	(net 14 "unconnected-(RV1-Pad3)")
 	(footprint "LED_THT:LED_D5.0mm"
 		(layer "F.Cu")
@@
 			(layers "*.Cu" "*.Mask")
 			(remove_unused_layers no)
-			(net 10 "VSS")
+			(net 14 "unconnected-(RV1-Pad3)")
 			(pinfunction "3")
-			(pintype "passive")
+			(pintype "passive+no_connect")
 		)
 		(embedded_fonts no)
@@
 		(layer "B.SilkS")
 	)
-	(gr_poly
-		(pts
-			(xy 188.126882 86.231699) (xy 188.115273 86.232582) (xy 188.103832 86.234035) (xy 188.092575 86.236046)
-			(xy 188.081515 86.238598) (xy 188.070667 86.241679) (xy 188.060046 86.245273) (xy 188.049665 86.249366)
-			(xy 188.039538 86.253944) (xy 188.029682 86.258992) (xy 188.020109 86.264496) (xy 188.010834 86.270443)
-			(xy 188.001871 86.276816) (xy 187.993235 86.283602) (xy 187.984941 86.290787) (xy 187.977001 86.298357)
-			(xy 187.969432 86.306296) (xy 187.962247 86.31459) (xy 187.955461 86.323226) (xy 187.949087 86.332189)
-			(xy 187.943141 86.341464) (xy 187.937637 86.351037) (xy 187.932589 86.360893) (xy 187.928011 86.37102)
-			(xy 187.923917 86.381401) (xy 187.920324 86.392022) (xy 187.917243 86.40287) (xy 187.91469 86.41393)
-			(xy 187.91268 86.425187) (xy 187.911226 86.436628) (xy 187.910344 86.448237) (xy 187.910046 86.460001)
-			(xy 187.910344 86.471765) (xy 187.911226 86.483374) (xy 187.91268 86.494814) (xy 187.91469 86.506072)
-			(xy 187.917243 86.517132) (xy 187.920324 86.527979) (xy 187.923917 86.538601) (xy 187.928011 86.548982)
-			(xy 187.932589 86.559108) (xy 187.937637 86.568965) (xy 187.943141 86.578538) (xy 187.949087 86.587813)
-			(xy 187.955461 86.596776) (xy 187.962247 86.605412) (xy 187.969432 86.613706) (xy 187.977001 86.621645)
-			(xy 187.984941 86.629214) (xy 187.993235 86.636399) (xy 188.001871 86.643186) (xy 188.010834 86.649559)
-			(xy 188.020109 86.655505) (xy 188.029682 86.66101) (xy 188.039538 86.666058) (xy 188.049665 86.670636)
-			(xy 188.060046 86.674729) (xy 188.070667 86.678323) (xy 188.081515 86.681404) (xy 188.092575 86.683956)
-			(xy 188.103832 86.685966) (xy 188.115273 86.68742) (xy 188.126882 86.688303) (xy 188.138646 86.6886)
-			(xy 188.15041 86.688303) (xy 188.162019 86.68742) (xy 188.173459 86.685966) (xy 188.184717 86.683956)
-			(xy 188.195777 86.681404) (xy 188.206625 86.678323) (xy 188.217246 86.674729) (xy 188.227627 86.670636)
-			(xy 188.237753 86.666058) (xy 188.24761 86.66101) (xy 188.257183 86.655505) (xy 188.266458 86.649559)
-			(xy 188.275421 86.643186) (xy 188.284057 86.636399) (xy 188.292351 86.629214) (xy 188.300291 86.621645)
-			(xy 188.30786 86.613706) (xy 188.315045 86.605412) (xy 188.321831 86.596776) (xy 188.328205 86.587813)
-			(xy 188.334151 86.578538) (xy 188.339655 86.568965) (xy 188.344703 86.559108) (xy 188.349281 86.548982)
-			(xy 188.353375 86.538601) (xy 188.356969 86.527979) (xy 188.360049 86.517132) (xy 188.362602 86.506072)
-			(xy 188.364612 86.494814) (xy 188.366066 86.483374) (xy 188.366948 86.471765) (xy 188.367246 86.460001)
-			(xy 188.366948 86.448237) (xy 188.366066 86.436628) (xy 188.364612 86.425187) (xy 188.362602 86.41393)
-			(xy 188.360049 86.40287) (xy 188.356969 86.392022) (xy 188.353375 86.381401) (xy 188.349281 86.37102)
-			(xy 188.344703 86.360893) (xy 188.339655 86.351037) (xy 188.334151 86.341464) (xy 188.328205 86.332189)
-			(xy 188.321831 86.323226) (xy 188.315045 86.31459) (xy 188.30786 86.306296) (xy 188.300291 86.298357)
-			(xy 188.292351 86.290787) (xy 188.284057 86.283602) (xy 188.275421 86.276816) (xy 188.266458 86.270443)
-			(xy 188.257183 86.264496) (xy 188.24761 86.258992) (xy 188.237753 86.253944) (xy 188.227627 86.249366)
-			(xy 188.217246 86.245273) (xy 188.206625 86.241679) (xy 188.195777 86.238598) (xy 188.184717 86.236046)
-			(xy 188.173459 86.234035) (xy 188.162019 86.232582) (xy 188.15041 86.231699) (xy 188.138646 86.231401)
-		)
-		(stroke
-			(width 0.076199)
-			(type solid)
-		)
-		(fill yes)
-		(layer "B.SilkS")
-	)
 	(gr_line
 		(start 176.501899 90.559747)
@@
 	)
 	(gr_line
-		(start 188.138646 86.46)
-		(end 179.883647 86.46)
-		(stroke
-			(width 0.076199)
-			(type solid)
-		)
-		(layer "B.SilkS")
-	)
-	(gr_line
 		(start 182.169646 80.11)
 		(end 181.788646 79.475)
@@
 	)
 	(segment
-		(start 160.06 116.46)
-		(end 170.06 116.46)
-		(width 0.2)
-		(layer "B.Cu")
-		(net 10)
-	)
-	(segment
 		(start 149.351 116.449)
 		(end 160.049 116.449)
@@
 			"ca59d706-841b-4ae6-ba90-7d17d9bf56c2" "caa50c19-c404-4505-b1c1-c8157f1b222b"
 			"caa62cc0-cc3e-43fb-a819-188651f954aa" "cab258ca-6422-4dbd-a0ad-1988b39e39a4"
-			"caba611f-248b-4ab5-ab23-ce22eb0eb74f" "cacce20f-5d34-4578-9076-f63f4bf3259b"
-			"cb2b0908-2bac-4bf2-beec-c21f9bba9a31" "cb393b5e-d40e-490c-a413-564ea272278f"
-			"cb534c5b-8e08-457e-b98e-2b9eb4fa639d" "cb576a45-3906-4b27-a875-caa7b461df23"
-			"cb6d34a9-4f58-4505-9c64-54679800bbff" "cb7109d8-37f6-46ca-9a8c-3bd9ef70f7be"
-			"cb80caa0-e0da-4f35-825e-0e7e7a33ba1f" "cb8bdc88-357e-4d3e-831a-3a8e7d875659"
-			"cbac68ed-415b-4987-a1f9-d801844f87bd" "cbf039f1-4b35-4cb1-aee3-d8c2e9c72919"
-			"cc21641c-fdad-4601-85c7-ac5c9edfc55a" "ccb57afb-3349-4861-9635-bcee63d28471"
-			"ccb7f019-8458-4857-aa1b-696479797f0c" "cce53369-6a31-4254-b3c5-bf386e8ff28a"
-			"cce7b4bf-d2a4-49d2-b38b-aa152a767b88" "cce8e610-9ce8-49ad-8c8f-def5d1ad5c12"
-			"ccfbf2c6-db72-41a2-beb5-c71b9fbf08a2" "cd28b1dd-db85-4995-8db9-dc88d490cabc"
-			"cd38d962-ef07-451d-b4db-754f9d9a6e2d" "cd3a2e47-2d9f-4643-bdb5-fa93d2f99c7a"
-			"cd4217ae-b4d7-4eeb-9be9-598f1add5446" "cd52aea4-c5f9-4720-b73d-59dee7fc61e1"
-			"cd606add-ce5a-4980-aff2-a60ae2f4b874" "cd756708-b2a6-436b-8be8-4152e95d9372"
-			"cd761bfb-9943-4944-bf88-6fb98f022bcd" "cd8c28d4-8808-4c74-adc6-95a62a72a3e2"
-			"cdae90c5-4718-41a0-adcc-f975d8e73f64" "cdb705c6-17fb-4ab7-969c-ab3e5418474f"
-			"cde51d74-df7a-4952-992d-e2808219fc84" "cde716da-553c-442b-8ca0-064f853710ba"
-			"ce1378cf-8319-4e50-ac04-fab2cecb5afd" "ce184821-12cf-4f28-9d93-b59ebccb3956"
-			"ce29f92a-a01f-4307-98a0-2f8930506c00" "ce3f9261-c729-4102-b5ea-f82d73de39aa"
-			"ce5d2797-78c1-4948-b3ab-63c19715748c" "ce84b474-1c9a-43bb-bf36-2e05ec2f1f00"
-			"ce879061-bb9b-4dd6-9d1e-3909b53873ab" "ced6f007-07bf-4703-b533-d19f69c7aa2c"
-			"ceeb1d9d-ed69-407b-b0bc-4ebde3e7fd83" "cf3c3a1a-6302-4228-bda1-6bf910ee64ab"
-			"cf59cf64-d6f9-4525-b44f-8633d7a82758" "cf7f303d-9b8c-4057-a2d6-bf751eaf6d42"
-			"cf8517af-f098-40e9-b97b-ced0c191386e" "cfd18772-b661-4956-91ca-1da2ab859893"
-			"cfd240ea-a0d9-4d8b-b481-fc984274fe51" "cfef0c76-5f67-4adf-b468-4ae7f10d8163"
-			"cfff20e3-34b6-42cf-897c-cf3e1c0f780b" "d0250e23-3803-49c0-8ae6-d3caa4c8aa73"
-			"d038c14f-c301-41df-a5cd-fdba2a14b72d" "d0594df0-b353-4ee9-b8c7-f1de6464f0d3"
-			"d06294ad-028f-4b38-a31b-6b59e39bb710" "d0a03490-f9ae-427b-8b69-28cd45e662c8"
-			"d0a30d7e-2d6c-4caa-8816-1cf8e007f1f3" "d0aeb347-97a3-4ad1-be18-902949d8d897"
-			"d11bcf19-8d70-4dab-a3ad-8a355ec7f55e" "d1223cff-1d63-49b0-9555-b6db9a93afc9"
+			"cacce20f-5d34-4578-9076-f63f4bf3259b" "cb2b0908-2bac-4bf2-beec-c21f9bba9a31"
+			"cb393b5e-d40e-490c-a413-564ea272278f" "cb534c5b-8e08-457e-b98e-2b9eb4fa639d"
+			"cb576a45-3906-4b27-a875-caa7b461df23" "cb6d34a9-4f58-4505-9c64-54679800bbff"
+			"cb7109d8-37f6-46ca-9a8c-3bd9ef70f7be" "cb80caa0-e0da-4f35-825e-0e7e7a33ba1f"
+			"cb8bdc88-357e-4d3e-831a-3a8e7d875659" "cbac68ed-415b-4987-a1f9-d801844f87bd"
+			"cbf039f1-4b35-4cb1-aee3-d8c2e9c72919" "cc21641c-fdad-4601-85c7-ac5c9edfc55a"
+			"ccb57afb-3349-4861-9635-bcee63d28471" "ccb7f019-8458-4857-aa1b-696479797f0c"
+			"cce53369-6a31-4254-b3c5-bf386e8ff28a" "cce7b4bf-d2a4-49d2-b38b-aa152a767b88"
+			"cce8e610-9ce8-49ad-8c8f-def5d1ad5c12" "ccfbf2c6-db72-41a2-beb5-c71b9fbf08a2"
+			"cd28b1dd-db85-4995-8db9-dc88d490cabc" "cd38d962-ef07-451d-b4db-754f9d9a6e2d"
+			"cd3a2e47-2d9f-4643-bdb5-fa93d2f99c7a" "cd4217ae-b4d7-4eeb-9be9-598f1add5446"
+			"cd52aea4-c5f9-4720-b73d-59dee7fc61e1" "cd606add-ce5a-4980-aff2-a60ae2f4b874"
+			"cd756708-b2a6-436b-8be8-4152e95d9372" "cd761bfb-9943-4944-bf88-6fb98f022bcd"
+			"cd8c28d4-8808-4c74-adc6-95a62a72a3e2" "cdae90c5-4718-41a0-adcc-f975d8e73f64"
+			"cdb705c6-17fb-4ab7-969c-ab3e5418474f" "cde51d74-df7a-4952-992d-e2808219fc84"
+			"cde716da-553c-442b-8ca0-064f853710ba" "ce1378cf-8319-4e50-ac04-fab2cecb5afd"
+			"ce184821-12cf-4f28-9d93-b59ebccb3956" "ce29f92a-a01f-4307-98a0-2f8930506c00"
+			"ce3f9261-c729-4102-b5ea-f82d73de39aa" "ce5d2797-78c1-4948-b3ab-63c19715748c"
+			"ce84b474-1c9a-43bb-bf36-2e05ec2f1f00" "ce879061-bb9b-4dd6-9d1e-3909b53873ab"
+			"ced6f007-07bf-4703-b533-d19f69c7aa2c" "ceeb1d9d-ed69-407b-b0bc-4ebde3e7fd83"
+			"cf3c3a1a-6302-4228-bda1-6bf910ee64ab" "cf59cf64-d6f9-4525-b44f-8633d7a82758"
+			"cf7f303d-9b8c-4057-a2d6-bf751eaf6d42" "cf8517af-f098-40e9-b97b-ced0c191386e"
+			"cfd18772-b661-4956-91ca-1da2ab859893" "cfd240ea-a0d9-4d8b-b481-fc984274fe51"
+			"cfef0c76-5f67-4adf-b468-4ae7f10d8163" "cfff20e3-34b6-42cf-897c-cf3e1c0f780b"
+			"d0250e23-3803-49c0-8ae6-d3caa4c8aa73" "d038c14f-c301-41df-a5cd-fdba2a14b72d"
+			"d0594df0-b353-4ee9-b8c7-f1de6464f0d3" "d06294ad-028f-4b38-a31b-6b59e39bb710"
+			"d0a03490-f9ae-427b-8b69-28cd45e662c8" "d0a30d7e-2d6c-4caa-8816-1cf8e007f1f3"
+			"d0aeb347-97a3-4ad1-be18-902949d8d897" "d11bcf19-8d70-4dab-a3ad-8a355ec7f55e"
 			"d13a746d-793e-4ae5-bee9-ad1639aeed48" "d1741d8f-b5e8-402d-bbe8-4d2d2a7d3202"
 			"d1769cd7-e158-4284-bf5f-92e5404ecfd7" "d18c726f-01e7-4b72-83f0-df0ce3c9676c"
