File: lightup-namebadge.kicad_pcb (KiCad board)
At the start: 2 copper layers, 100 x 50 mm, 26 parts, among them Q1 PNP, Q2 NPN, Q3 NPN, Q4 NPN, Q5 NPN, SW1 SW_Push, SW2 SW_Push

Commit message: fix: new resistor values and more thermal relif for battery connector
Parts:
- R6: value 220 -> 680
- RV1, RV2: value 100k -> 5k
- moved R6 7.60 mm to (136.4, 115.5), turned to 0 degrees
Connections:
- Q2 pad 3: Net-(Q2-E) -> LEDS_INPUT
- R1 pad 1: Net-(Q1-B) -> Net-(R1-Pad1)
- R6 pad 1: Net-(Q2-E) -> Net-(R1-Pad1)
- R6 pad 2: LEDS_INPUT -> Net-(Q1-B)
- RV2 pad 3: VSS -> unconnected-(RV2-Pad3)
Routing:
- net VSS: track 70.5 -> 41.5 mm
- net Net-(Q3-B): track 62.4 -> 39.7 mm
- net Net-(R1-Pad1): track 0.00 -> 17.0 mm
- net VDD: track 0.00 -> 15.9 mm
- net Net-(Q1-E): track 40.4 -> 51.3 mm
- net Net-(Q4-C): track 23.6 -> 32.7 mm
- net Net-(Q1-B): track 22.6 -> 14.1 mm
- net Net-(Q5-B): track 82.4 -> 74.1 mm
- net Net-(Q2-E): track 6.11 -> 0.00 mm, vias 1 -> 0
- net Net-(Q4-B): track 96.8 -> 92.7 mm
- net LEDS_INPUT: track 141.5 -> 144.4 mm
Other:
- board text added: "2025_06_20"
